Commit message: Update robot with kinect and RGBD Cameras

File: urdf/fouliex_bot.xacro (robot description, xacro)
@@ -134,28 +134,86 @@
     </joint>
     <!-- Camera Link -->
-    <link name='camera'>
-        <inertial>
-            <mass value="0.1"/>
-            <origin xyz="0.0 0 0" rpy=" 0 0 0"/>
-            <inertia ixx="1e-6" ixy="0" ixz="0" iyy="1e-6" iyz="0" izz="1e-6"/>
-        </inertial>
-        <collision name='collision'>
-            <origin xyz="0.0 0 0" rpy=" 0 0 0"/>
-            <geometry>
-                <box size="0.05 0.05 0.05"/>
-            </geometry>
-        </collision>
-        <visual name='camera_visual'>
-            <origin xyz="0.0 0 0" rpy=" 0 0 0"/>
-            <geometry>
-                <box size="0.05 0.05 0.05"/>
-            </geometry>
-        </visual>
+    <link name="camera">
+        <inertial>
+            <mass value="0.01" />
+            <origin xyz="0 0 0" />
+            <inertia ixx="0.001" ixy="0.0" ixz="0.0"
+                     iyy="0.001" iyz="0.0"
+                     izz="0.001" />
+        </inertial>
+        <visual>
+            <origin xyz=" 0 0 0 " rpy="0 0 0" />
+            <geometry>
+                <mesh filename="package://fouliex_bot/meshes/kinect.dae"/>
+            </geometry>
+        </visual>
+        <collision>
+            <origin xyz="0.0 0.0 0.0" rpy="0 0 0" />
+            <geometry>
+                <box size="0.0730 .2760 0.0720"/>
+            </geometry>
+        </collision>
+    </link>
+    <joint name="camera_depth_joint" type="fixed">
+        <origin xyz="0 0.011 0" rpy="0 0 0" />
+        <parent link="camera" />
+        <child link="camera_depth_frame" />
+    </joint>
+    <link name="camera_depth_frame">
+        <inertial>
+            <mass value="0.01" />
+            <origin xyz="0 0 0" />
+            <inertia ixx="0.001" ixy="0.0" ixz="0.0"
+                     iyy="0.001" iyz="0.0"
+                     izz="0.001" />
+        </inertial>
+    </link>
+    <joint name="camera_depth_optical_joint" type="fixed">
+        <origin xyz="0 0 0" rpy="-1.57 0 1.57" />
+        <parent link="camera_depth_frame" />
+        <child link="camera_depth_optical_frame" />
+    </joint>
+    <link name="camera_depth_optical_frame">
+        <inertial>
+            <mass value="0.001" />
+            <origin xyz="0 0 0" />
+            <inertia ixx="0.0001" ixy="0.0" ixz="0.0"
+                     iyy="0.0001" iyz="0.0"
+                     izz="0.0001" />
+        </inertial>
+    </link>
+    <joint name="camera_rgb_joint" type="fixed">
+        <origin xyz="0 -0.012 0" rpy="0 0 0" />
+        <parent link="camera" />
+        <child link="camera_rgb_frame" />
+    </joint>
+    <link name="camera_rgb_frame">
+        <inertial>
+            <mass value="0.001" />
+            <origin xyz="0 0 0" />
+            <inertia ixx="0.0001" ixy="0.0" ixz="0.0"
+                     iyy="0.0001" iyz="0.0"
+                     izz="0.0001" />
+        </inertial>
+    </link>
+    <joint name="camera_rgb_optical_joint" type="fixed">
+        <origin xyz="0 0 0" rpy="-1.57 0 1.57" />
+        <parent link="camera_rgb_frame" />
+        <child link="camera_rgb_optical_frame" />
+    </joint>
+    <link name="camera_rgb_optical_frame">
+        <inertial>
+            <mass value="0.001" />
+            <origin xyz="0 0 0" />
+            <inertia ixx="0.0001" ixy="0.0" ixz="0.0"
+                     iyy="0.0001" iyz="0.0"
+                     izz="0.0001" />
+        </inertial>
     </link>
     <!-- Camera Joint -->
-    <joint type="fixed" name="camera_joint">
-        <origin xyz="0.2 0 0" rpy="0 0 0"/>
-        <child link="camera"/>
-        <parent link="chassis"/>
+    <joint name="base_camera_joint" type="fixed">
+        <origin xyz="0.22 0 0" rpy="0 -0.349 0" />
+        <parent link="chassis" />
+        <child link="camera" />
     </joint>
     <!-- Laser RangeFinder(hokuyo) Link -->

Commit message: Add Pictures

File: urdf/fouliex_bot.xacro (robot description, xacro)
@@ -170,5 +170,5 @@
     </link>
     <joint name="camera_depth_optical_joint" type="fixed">
-        <origin xyz="0 0 0" rpy="-1.57 0 1.57" />
+        <origin xyz="0 0 0" rpy="-1.57 0 -1.57" />
         <parent link="camera_depth_frame" />
         <child link="camera_depth_optical_frame" />
@@ -198,5 +198,5 @@
     </link>
     <joint name="camera_rgb_optical_joint" type="fixed">
-        <origin xyz="0 0 0" rpy="-1.57 0 1.57" />
+        <origin xyz="0 0 0" rpy="-1.57 0 -1.57" />
         <parent link="camera_rgb_frame" />
         <child link="camera_rgb_optical_frame" />
